File: Out_8x10/Hi8.kicad_sch (KiCad schematic)
At the start: 59 parts, among them J5 Conn_01x09, J6 Conn_01x10, Q1 2N7002, Q10 AO3401A, Q11 AO3401A, Q12 AO3401A, Q13 2N7002, Q14 2N7002, Q15 AO3401A, Q16 AO3401A, Q2 2N7002, Q3 2N7002, Q4 AO3401A, Q5 AO3401A, Q6 AO3401A, Q7 2N7002, Q8 2N7002, Q9 2N7002, U10 L78L24_SOT89, U11 L78L24_SOT89, U12 L78L24_SOT89, U13 L78L24_SOT89, U6 L78L24_SOT89, U7 L78L24_SOT89, U8 L78L24_SOT89, U9 L78L24_SOT89

Commit message: V1.0.0
Parts:
- C41: JLCPCB Rotation Offset (none) -> 180
Other:
- title: High Side Switches -> Out_8x10
Changed lines of the file:
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@@
   (paper "A4")
   (title_block
-    (title "High Side Switches")
-    (date "2023-10-08")
-    (rev "0.2.0")
+    (title "Out_8x10")
+    (date "2024-12-01")
+    (rev "1.0.0")
   )
   (junction (at 173.99 132.08) (diameter 0) (color 0 0 0 0)
@@
       (effects (font (size 1.27 1.27)) hide)
     )
+    (property "JLCPCB Rotation Offset" "180" (id 4) (at 33.02 175.26 0)
+      (effects (font (size 1.27 1.27)) hide)
+    )
