File: Out_8x10/Lo10.kicad_sch (KiCad schematic)
At the start: 32 parts, among them J7 Conn_01x09, J8 Conn_01x12, Q17 AO3400A, Q18 AO3400A, Q19 AO3400A, Q20 AO3400A, Q21 AO3400A, Q22 AO3400A, Q23 AO3400A, Q24 AO3400A, Q25 AO3400A, Q26 AO3400A

Commit message: V1.0.0
Other:
- title: Low Side Switches -> Out_8x10
Changed lines of the file:
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@@
   (paper "A4")
   (title_block
-    (title "Low Side Switches")
-    (date "2023-10-08")
-    (rev "0.2.0")
+    (title "Out_8x10")
+    (date "2024-12-01")
+    (rev "1.0.0")
   )
   (junction (at 45.72 68.58) (diameter 0) (color 0 0 0 0)
